Commit message: Unit 2: 2.4 Update the robot description file

File: ros2_control/unit2/rrbot_unit2/urdf/rrbot.xacro (robot description, xacro)
@@ -169,3 +169,24 @@
   </joint>
   <link name="camera_link_optical"></link>
+  <ros2_control name="MyRobotSystem" type="system">
+    <hardware>
+      <plugin>gazebo_ros2_control/GazeboSystem</plugin>
+    </hardware>
+    <joint name="joint1">
+      <command_interface name="position">
+        <param name="min">-6.28</param>
+        <param name="max">6.28</param>
+      </command_interface>
+      <state_interface name="position"/>
+      <state_interface name="velocity"/>
+      <state_interface name="effort"/>
+    </joint>
+  </ros2_control>
+  <!-- Gazebo's ros2_control plugin -->
+  <gazebo>
+    <plugin filename="libgazebo_ros2_control.so" name="gazebo_ros2_control">
+      <robot_sim_type>gazebo_ros2_control/GazeboSystem</robot_sim_type>
+      <parameters>$(find my_robot_bringup)/config/controller_configuration.yaml</parameters>
+    </plugin>
+  </gazebo>
 </robot>

Commit message: Unit 2: 2.7 Apply your learning

File: ros2_control/unit2/rrbot_unit2/urdf/rrbot.xacro (robot description, xacro)
@@ -169,9 +169,18 @@
   </joint>
   <link name="camera_link_optical"></link>
-  <ros2_control name="MyRobotSystem" type="system">
+  <ros2_control name="GazeboSystem" type="system">
     <hardware>
       <plugin>gazebo_ros2_control/GazeboSystem</plugin>
     </hardware>
     <joint name="joint1">
+      <command_interface name="position">
+        <param name="min">-6.28</param>
+        <param name="max">6.28</param>
+      </command_interface>
+      <state_interface name="position"/>
+      <state_interface name="velocity"/>
+      <state_interface name="effort"/>
+    </joint>
+    <joint name="joint2">
       <command_interface name="position">
         <param name="min">-6.28</param>
