Commit message: Unit 4: 4.17  Switching the Hardware Plugin

File: ros2_control_course/unit3/rrbot_unit3/urdf/rrbot.xacro (robot description, xacro)
@@ -169,3 +169,25 @@
   </joint>
   <link name="camera_link_optical"></link>
+  <ros2_control name="DemoHardware" type="system">
+      <hardware>
+        <plugin>my_robot_hardware_interface/RRBotSystemPositionOnlyHardware</plugin>
+        <param name="example_param_hw_start_duration_sec">0.0</param>
+        <param name="example_param_hw_stop_duration_sec">3.0</param>
+        <param name="example_param_hw_slowdown">10.0</param>
+      </hardware>
+      <joint name="joint1">
+        <command_interface name="position">
+          <param name="min">-1</param>
+          <param name="max">1</param>
+        </command_interface>
+        <state_interface name="position"/>
+      </joint>
+      <joint name="joint2">
+        <command_interface name="position">
+          <param name="min">-1</param>
+          <param name="max">1</param>
+        </command_interface>
+        <state_interface name="position"/>
+      </joint>
+    </ros2_control>
 </robot>
