Commit message: Unit 5: 5.19 Switching the Hardware Plugin

File: ros2_control_course/unit4/rrbot_unit4/urdf/rrbot.xacro (robot description, xacro)
@@ -169,3 +169,27 @@
   </joint>
   <link name="camera_link_optical"></link>
+    <ros2_control name="DynamixelHardware" type="system">
+      <hardware>
+        <plugin>dynamixel_hardware/DynamixelHardware</plugin>
+        <param name="usb_port">/dev/ttyUSB0</param>
+        <param name="baud_rate">1000000</param>
+        <param name="use_dummy">true</param>
+      </hardware>
+      <joint name="joint1">
+        <param name="id">11</param>
+        <command_interface name="position"/>
+        <command_interface name="velocity"/>
+        <state_interface name="position"/>
+        <state_interface name="velocity"/>
+        <state_interface name="effort"/>
+      </joint>
+      <joint name="joint2">
+        <param name="id">12</param>
+        <command_interface name="position"/>
+        <command_interface name="velocity"/>
+        <state_interface name="position"/>
+        <state_interface name="velocity"/>
+        <state_interface name="effort"/>
+      </joint>
+    </ros2_control>
 </robot>
