Commit message: Unit 6.3 The effort_controllers

File: ros2_control_course/unit5/rrbot_unit5/urdf/rrbot.xacro (robot description, xacro)
@@ -170,4 +170,32 @@
   <link name="camera_link_optical"></link>
 <!-- place your ros2_control XML tags below this line -->
+  <ros2_control name="effort_controllers_exercise" type="system">
+    <hardware>
+      <plugin>gazebo_ros2_control/GazeboSystem</plugin>
+    </hardware>
+    <joint name="joint1">
+      <command_interface name="effort">
+        <param name="min">-1000</param>
+        <param name="max">1000</param>
+      </command_interface>
+      <state_interface name="position"/>
+      <state_interface name="velocity"/>
+      <state_interface name="effort"/>
+    </joint>
+    <joint name="joint2">
+      <command_interface name="effort">
+        <param name="min">-1000</param>
+        <param name="max">1000</param>
+      </command_interface>
+      <state_interface name="position"/>
+      <state_interface name="velocity"/>
+      <state_interface name="effort"/>
+    </joint>
+  </ros2_control>
+  <gazebo>
+    <plugin filename="libgazebo_ros2_control.so" name="gazebo_ros2_control">
+      <parameters>$(find rrbot_unit5)/config/effort_controller_config.yaml</parameters>
+    </plugin>
+  </gazebo>
 <!-- place your ros2_control XML tags above this line -->
 </robot>

Commit message: Unit 6: 6.4 The velocity_controllers

File: ros2_control_course/unit5/rrbot_unit5/urdf/rrbot.xacro (robot description, xacro)
@@ -170,30 +170,30 @@
   <link name="camera_link_optical"></link>
 <!-- place your ros2_control XML tags below this line -->
-  <ros2_control name="effort_controllers_exercise" type="system">
+    <ros2_control name="velocity_controller_exercise" type="system">
     <hardware>
       <plugin>gazebo_ros2_control/GazeboSystem</plugin>
     </hardware>
-    <joint name="joint1">
-      <command_interface name="effort">
-        <param name="min">-1000</param>
-        <param name="max">1000</param>
-      </command_interface>
-      <state_interface name="position"/>
-      <state_interface name="velocity"/>
-      <state_interface name="effort"/>
-    </joint>
-    <joint name="joint2">
-      <command_interface name="effort">
-        <param name="min">-1000</param>
-        <param name="max">1000</param>
-      </command_interface>
-      <state_interface name="position"/>
-      <state_interface name="velocity"/>
-      <state_interface name="effort"/>
-    </joint>
-  </ros2_control>
+      <joint name="joint1">
+        <command_interface name="velocity">
+          <param name="min">-1</param>
+          <param name="max">1</param>
+        </command_interface>
+        <state_interface name="position"/>
+        <state_interface name="velocity"/>
+        <state_interface name="acceleration"/>
+      </joint>
+      <joint name="joint2">
+        <command_interface name="velocity">
+          <param name="min">-1</param>
+          <param name="max">1</param>
+        </command_interface>
+        <state_interface name="position"/>
+        <state_interface name="velocity"/>
+        <state_interface name="acceleration"/>
+      </joint>
+    </ros2_control>
   <gazebo>
     <plugin filename="libgazebo_ros2_control.so" name="gazebo_ros2_control">
-      <parameters>$(find rrbot_unit5)/config/effort_controller_config.yaml</parameters>
+      <parameters>$(find rrbot_unit5)/config/velocity_controller_config.yaml</parameters>
     </plugin>
   </gazebo>

Commit message: Unit 6: 6.2 The position_controllers (Add ros2 control in xacro)

File: ros2_control_course/unit5/rrbot_unit5/urdf/rrbot.xacro (robot description, xacro)
@@ -170,30 +170,30 @@
   <link name="camera_link_optical"></link>
 <!-- place your ros2_control XML tags below this line -->
-    <ros2_control name="velocity_controller_exercise" type="system">
+  <ros2_control name="position_controllers_exercise" type="system">
     <hardware>
       <plugin>gazebo_ros2_control/GazeboSystem</plugin>
     </hardware>
-      <joint name="joint1">
-        <command_interface name="velocity">
-          <param name="min">-1</param>
-          <param name="max">1</param>
-        </command_interface>
-        <state_interface name="position"/>
-        <state_interface name="velocity"/>
-        <state_interface name="acceleration"/>
-      </joint>
-      <joint name="joint2">
-        <command_interface name="velocity">
-          <param name="min">-1</param>
-          <param name="max">1</param>
-        </command_interface>
-        <state_interface name="position"/>
-        <state_interface name="velocity"/>
-        <state_interface name="acceleration"/>
-      </joint>
-    </ros2_control>
+    <joint name="joint1">
+      <command_interface name="position">
+        <param name="min">-1000</param>
+        <param name="max">1000</param>
+      </command_interface>
+      <state_interface name="position"/>
+      <state_interface name="velocity"/>
+      <state_interface name="effort"/>
+    </joint>
+    <joint name="joint2">
+      <command_interface name="position">
+        <param name="min">-1000</param>
+        <param name="max">1000</param>
+      </command_interface>
+      <state_interface name="position"/>
+      <state_interface name="velocity"/>
+      <state_interface name="effort"/>
+    </joint>
+  </ros2_control>
   <gazebo>
     <plugin filename="libgazebo_ros2_control.so" name="gazebo_ros2_control">
-      <parameters>$(find rrbot_unit5)/config/velocity_controller_config.yaml</parameters>
+      <parameters>$(find rrbot_unit5)/config/position_controller_config.yaml</parameters>
     </plugin>
   </gazebo>

Commit message: Unit 6: 6.5 The forward_command_controller

File: ros2_control_course/unit5/rrbot_unit5/urdf/rrbot.xacro (robot description, xacro)
@@ -170,30 +170,47 @@
   <link name="camera_link_optical"></link>
 <!-- place your ros2_control XML tags below this line -->
-  <ros2_control name="position_controllers_exercise" type="system">
+  <ros2_control name="forward_command_controllers_exercise" type="system">
     <hardware>
       <plugin>gazebo_ros2_control/GazeboSystem</plugin>
     </hardware>
-    <joint name="joint1">
-      <command_interface name="position">
-        <param name="min">-1000</param>
-        <param name="max">1000</param>
-      </command_interface>
-      <state_interface name="position"/>
-      <state_interface name="velocity"/>
-      <state_interface name="effort"/>
-    </joint>
-    <joint name="joint2">
-      <command_interface name="position">
-        <param name="min">-1000</param>
-        <param name="max">1000</param>
-      </command_interface>
-      <state_interface name="position"/>
-      <state_interface name="velocity"/>
-      <state_interface name="effort"/>
-    </joint>
+      <joint name="joint1">
+          <command_interface name="position">
+          <param name="min">-1</param>
+          <param name="max">1</param>
+        </command_interface>
+        <command_interface name="velocity">
+          <param name="min">-1</param>
+          <param name="max">1</param>
+        </command_interface>
+        <command_interface name="acceleration">
+          <param name="min">-1</param>
+          <param name="max">1</param>
+        </command_interface>
+        <state_interface name="position"/>
+        <state_interface name="velocity"/>
+        <state_interface name="acceleration"/>
+      </joint>
+      <joint name="joint2">
+          <command_interface name="position">
+          <param name="min">-1</param>
+          <param name="max">1</param>
+        </command_interface>
+        <command_interface name="velocity">
+          <param name="min">-1</param>
+          <param name="max">1</param>
+        </command_interface>
+        <command_interface name="acceleration">
+          <param name="min">-1</param>
+          <param name="max">1</param>
+        </command_interface>
+        <state_interface name="position"/>
+        <state_interface name="velocity"/>
+        <state_interface name="acceleration"/>
+      </joint>
   </ros2_control>
   <gazebo>
     <plugin filename="libgazebo_ros2_control.so" name="gazebo_ros2_control">
-      <parameters>$(find rrbot_unit5)/config/position_controller_config.yaml</parameters>
+      <robot_sim_type>gazebo_ros2_control/GazeboSystem</robot_sim_type>
+      <parameters>$(find rrbot_unit5)/config/forward_command_controller_config.yaml</parameters>
     </plugin>
   </gazebo>

Commit message: Unit 6: 6.7 The diff_drive_controller

File: ros2_control_course/unit5/rrbot_unit5/urdf/rrbot.xacro (robot description, xacro)
@@ -170,18 +170,10 @@
   <link name="camera_link_optical"></link>
 <!-- place your ros2_control XML tags below this line -->
-  <ros2_control name="trajectory_controllers_exercise" type="system">
-    <hardware>
-      <plugin>gazebo_ros2_control/GazeboSystem</plugin>
-    </hardware>
-      <joint name="joint1">
-          <command_interface name="position">
-          <param name="min">-1</param>
-          <param name="max">1</param>
-        </command_interface>
+    <ros2_control name="diff_drive" type="system">
+      <hardware>
+          <plugin>gazebo_ros2_control/GazeboSystem</plugin>
+      </hardware>
+      <joint name="left_wheel_joint">
         <command_interface name="velocity">
-          <param name="min">-1</param>
-          <param name="max">1</param>
-        </command_interface>
-        <command_interface name="acceleration">
           <param name="min">-1</param>
           <param name="max">1</param>
@@ -189,16 +181,8 @@
         <state_interface name="position"/>
         <state_interface name="velocity"/>
-        <state_interface name="acceleration"/>
+        <state_interface name="effort"/>
       </joint>
-      <joint name="joint2">
-          <command_interface name="position">
-          <param name="min">-1</param>
-          <param name="max">1</param>
-        </command_interface>
+      <joint name="right_wheel_joint">
         <command_interface name="velocity">
-          <param name="min">-1</param>
-          <param name="max">1</param>
-        </command_interface>
-        <command_interface name="acceleration">
           <param name="min">-1</param>
           <param name="max">1</param>
@@ -206,14 +190,7 @@
         <state_interface name="position"/>
         <state_interface name="velocity"/>
-        <state_interface name="acceleration"/>
+        <state_interface name="effort"/>
       </joint>
-  </ros2_control>
-  <!-- Gazebo ros2_control plugin -->
-    <gazebo>
-    <plugin filename="libgazebo_ros2_control.so" name="gazebo_ros2_control">
-      <robot_sim_type>gazebo_ros2_control/GazeboSystem</robot_sim_type>
-      <parameters>$(find rrbot_unit5)/config/joint_trajectory_controller_config.yaml</parameters>
-    </plugin>
-  </gazebo>
+    </ros2_control>
 <!-- place your ros2_control XML tags above this line -->
 </robot>
